Commit message: working to eliminate undesirable gazebo7 behavior with PositionJointInterface

File: models/common.gazebo.xacro (robot description, xacro)
@@ -3,5 +3,8 @@
   <gazebo>
     <!-- turn on self-collision detection so that links will not pass through each other -->
-    <self_collide>1</self_collide>
+    <self_collide>0</self_collide>
+    <!-- disable the default behavior with PositionJointInterface that causes twists to be cleared -->
+    <!--preserveWorldVelocity>1</preserveWorldVelocity-->
+    <preserve_world_velocity>1</preserve_world_velocity>
     <!-- for the mobile base -->
     <!-- MQMX to (possibly?) replace this with ros control plugin -->

File: models/mobile_arm/mobile_arm.urdf.xacro (robot description, xacro)
@@ -8,4 +8,5 @@
   <xacro:include filename="$(find mobile_arm)/models/mobile_base/mobile_base.urdf.xacro"/>
   <!-- UR10 description -->
+  <!--xacro:include filename="$(find mobile_arm)/models/my_ur10/my_ur10.urdf.xacro" /-->
   <xacro:include filename="$(find ur_description)/urdf/ur10.urdf.xacro" />
   <xacro:ur10_robot prefix="" joint_limited="false"/>
@@ -16,3 +17,10 @@
     <child link="base_link" />
   </joint>
+  <!-- temp attach mobile base to ground -->
+  <!--link name="world" />
+  <joint name="world_joint" type="fixed">
+    <parent link="world" />
+    <child link = "chassis" />
+    <origin xyz="0.0 0.0 1.0" rpy="0.0 0.0 0.0" />
+  </joint-->
 </robot>

Commit message: created simple gripper with controller --- yet to add it to mobile arm

File: models/common.gazebo.xacro (robot description, xacro)
@@ -4,18 +4,4 @@
     <!-- turn on self-collision detection so that links will not pass through each other -->
     <self_collide>0</self_collide>
-    <!-- disable the default behavior with PositionJointInterface that causes twists to be cleared -->
-    <!--preserveWorldVelocity>1</preserveWorldVelocity-->
-    <preserve_world_velocity>1</preserve_world_velocity>
-    <!-- for the mobile base -->
-    <!-- MQMX to (possibly?) replace this with ros control plugin -->
-    <plugin name="differential_drive_controller" filename="libgazebo_ros_diff_drive.so">
-      <leftJoint>wheel_2_joint</leftJoint>
-      <rightJoint>wheel_5_joint</rightJoint>
-      <robotBaseFrame>chassis</robotBaseFrame>
-      <wheelSeparation>${chassis_width - wheel_thickness}</wheelSeparation>
-      <wheelDiameter>${2 * wheel_radius}</wheelDiameter>
-      <publishWheelJointState>true</publishWheelJointState>
-      <legacyMode>false</legacyMode>
-    </plugin>
     <!-- for the UR10, copied from $(find ur_description)/urdf/common.gazebo.xacro -->
     <plugin name="ros_control" filename="libgazebo_ros_control.so" />

File: models/mobile_arm/mobile_arm.urdf (robot description, URDF)
Before this commit: robot mobile_ur10, 17 links, 16 joints
Links:
- added link camera_link, mass 0.1; collision box size=0.1 0.1 0.1; visual box size=0.1 0.1 0.1
- added link gripper_link, mass 0.15; collision cylinder length=0.4 radius=0.15; visual cylinder length=0.4 radius=0.15
- added link mount_link, mass 0.15; collision box size=0.4 0.05 0.01; visual box size=0.4 0.05 0.01
Joints:
- added joint camera_to_mount: type fixed, parent mount_link, child camera_link, origin xyz=-.15 0 .055 rpy=0 0 0
- added joint gripper_to_mount: type fixed, parent mount_link, child gripper_link, origin xyz=.15 0 .205 rpy=0 0 0
- added joint mount_to_ur10: type fixed, parent tool0, child mount_link, origin xyz=0 0 .005 rpy=0 0 0
- joint shoulder_lift_joint: limit lower=-6.28318530718 upper=6.28318530718 effort=330.0 velocity=2.16 -> lower=-3.14159265359 upper=3.14159265359 effort=330.0 velocity=2.16
- joint shoulder_pan_joint: limit lower=-6.28318530718 upper=6.28318530718 effort=330.0 velocity=2.16 -> lower=-3.14159265359 upper=3.14159265359 effort=330.0 velocity=2.16
- joint wrist_1_joint: limit lower=-6.28318530718 upper=6.28318530718 effort=54.0 velocity=3.2 -> lower=-3.14159265359 upper=3.14159265359 effort=54.0 velocity=3.2
- joint wrist_2_joint: limit lower=-6.28318530718 upper=6.28318530718 effort=54.0 velocity=3.2 -> lower=-3.14159265359 upper=3.14159265359 effort=54.0 velocity=3.2
- joint wrist_3_joint: limit lower=-6.28318530718 upper=6.28318530718 effort=54.0 velocity=3.2 -> lower=-3.14159265359 upper=3.14159265359 effort=54.0 velocity=3.2

File: models/mobile_arm/mobile_arm.urdf.xacro (robot description, xacro)
@@ -3,6 +3,8 @@
        name="mobile_ur10">
   <!-- common Gazebo plugins and tags
-       note: there are also Gazebo tags in mobile_base.urdf.xacro to make the corner wheels frictionless -->
+       note: there are also Gazebo tags in mobile_base.urdf.xacro to make the corner wheels frictionless
+       note2: there are also Gazebo tags in mobile_base.urdf.xacro to configure the differential_drive_controller -->
   <xacro:include filename="$(find mobile_arm)/models/common.gazebo.xacro"/>
+  <!-- model descriptions -->
   <!-- mobile base description -->
   <xacro:include filename="$(find mobile_arm)/models/mobile_base/mobile_base.urdf.xacro"/>
@@ -10,5 +12,12 @@
   <!--xacro:include filename="$(find mobile_arm)/models/my_ur10/my_ur10.urdf.xacro" /-->
   <xacro:include filename="$(find ur_description)/urdf/ur10.urdf.xacro" />
-  <xacro:ur10_robot prefix="" joint_limited="false"/>
+  <xacro:ur10_robot prefix="" joint_limited="true"/>
+  <!-- mount for gripper and camera -->
+  <xacro:include filename="$(find mobile_arm)/models/mount_for_tool/mount_for_tool.urdf.xacro"/>
+  <!-- gripper -->
+  <xacro:include filename="$(find mobile_arm)/models/gripper/gripper.urdf.xacro"/>
+  <!-- camera -->
+  <xacro:include filename="$(find mobile_arm)/models/depth_camera/depth_camera.urdf.xacro"/>
+  <!-- joints for attaching models to each other -->
   <!-- joint to attach UR10 to mobile base -->
   <joint name="arm_to_mobile_base" type="fixed">
@@ -16,4 +25,22 @@
     <parent link="chassis" />
     <child link="base_link" />
+  </joint>
+  <!-- joint to attach mount for tool to UR10 -->
+  <joint name="mount_to_ur10" type="fixed">
+    <origin xyz="0 0 .005" rpy="0 0 0" />
+    <parent link="tool0" />
+    <child link="mount_link" />
+  </joint>
+  <!-- joint to attach gripper to mount -->
+  <joint name="gripper_to_mount" type="fixed">
+    <origin xyz=".15 0 .205" rpy="0 0 0" />
+    <parent link="mount_link" />
+    <child link="gripper_link" />
+  </joint>
+  <!-- joint to attach camera to mount -->
+  <joint name="camera_to_mount" type="fixed">
+    <origin xyz="-.15 0 .055" rpy="0 0 0" />
+    <parent link="mount_link" />
+    <child link="camera_link" />
   </joint>
   <!-- temp attach mobile base to ground -->
@@ -23,4 +50,4 @@
     <child link = "chassis" />
     <origin xyz="0.0 0.0 1.0" rpy="0.0 0.0 0.0" />
-  </joint-->
+    </joint-->
 </robot>

File: models/mobile_base/mobile_base.urdf.xacro (robot description, xacro)
@@ -122,3 +122,13 @@
   <xacro:make_wheel_n_frictionless n="4" />
   <xacro:make_wheel_n_frictionless n="6" />
+  <!-- MQMX to (possibly?) replace this with ros control plugin -->
+  <plugin name="differential_drive_controller" filename="libgazebo_ros_diff_drive.so">
+    <leftJoint>wheel_2_joint</leftJoint>
+    <rightJoint>wheel_5_joint</rightJoint>
+    <robotBaseFrame>chassis</robotBaseFrame>
+    <wheelSeparation>${chassis_width - wheel_thickness}</wheelSeparation>
+    <wheelDiameter>${2 * wheel_radius}</wheelDiameter>
+    <publishWheelJointState>true</publishWheelJointState>
+    <legacyMode>false</legacyMode>
+  </plugin>
 </robot>
